Commit message: urdf file is updated

File: imed_robot_update.urdf (robot description, URDF)
Before this commit: robot Robot, 9 links, 8 joints
Links:
- link base_link_prismatic: geometry visual mesh filename=/Users/kim/Documents/MATLAB/New Folder/path_planning/Basis_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 scale=1.00000000 1.00000000 1.00000000
- link link1: geometry collision box size=0.09000000 0.09000000 0.02000000; visual box size=0.03000000 0.0300000 0.02000000
- link link2: geometry collision box size=0.25230000 0.05000000 0.03100000; visual box size=0.25230000 0.05000000 0.03100000
- link link3: geometry collision box size=0.05000000 0.15560000 0.05000000; visual box size=0.05000000 0.15560000 0.05000000
- link link6: geometry collision box size=0.02000000 0.02000000 0.02000000; visual box size=0.02000000 0.02000000 0.02000000
- link tool: geometry collision mesh filename=SIEM_Spritze.stl scale=0.001000000 0.001000000 0.001000000; visual mesh filename=/Users/kim/Documents/MATLAB/New Folder/path_planning/SIEM_S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 scale=0.001000000 0.001000000 0.001000000
Joints:
- joint joint6: origin xyz=-0.03760000  0.00000000  0.03760000 rpy=-1.57079600  0.00000000  0.00000000 -> xyz=0  0.00000000  0.03760000 rpy=-1.57079600  0.00000000  0.00000000

Commit message: urdf issue is solved, however, the model is not equal to the real robot. But for collision detection is fair enough

File: imed_robot_update.urdf (robot description, URDF)
Before this commit: robot Robot, 9 links, 8 joints
Links:
- link link2: geometry collision box size=0.25230000 0.05000000 0.0200000; visual box size=0.25230000 0.05000000 0.0200000
- link link4: geometry collision box size=0.04000000 0.04450000 0.04000000; visual box size=0.04000000 0.04450000 0.04000000
- link link5: geometry collision box size=0.03760000 0.03760000 0.03760000; visual box size=0.03760000 0.037600000 0.03760000
Joints:
- joint joint5: origin xyz=0.00000000 0.00000000 0.04450000 rpy=1.57079600 0.00000000 0.00000000 -> xyz=0 -0.0225 0.0188 rpy=1.57079600 0.00000000 0.00000000
- joint joint6: origin xyz=0  0.00000000  0.03760000 rpy=-1.57079600  0.00000000  0.00000000 -> xyz=0  0.018800  0.01880000 rpy=-1.57079600  0.00000000  0.00000000

Commit message: modular edited 6

File: imed_robot_update.urdf (robot description, URDF)
Before this commit: robot Robot, 9 links, 8 joints
Links:
- link base_link_prismatic: geometry collision mesh filename=Basis_V5_scaled.stl scale=1.00000000 1.0000000 1.0000000; visual mesh filename=Basis_V5_scaled.stl scale=1.0000000 1.0000000 1.000000
- link tool: geometry collision mesh filename=SIEM_Spritze.stl scale=0.001000000 0.001000000 0.001000000; visual mesh filename=SIEM_Spritze.stl scale=0.001000000 0.001000000 0.001000000

Commit message: modular edited 6

File: imed_robot_update.urdf (robot description, URDF)
Before this commit: robot Robot, 9 links, 8 joints
Links:
- link base_link_prismatic: geometry collision mesh filename=Basis_V5_scaled.stl scale=0.001000000 0.00100000 0.00100000; visual mesh filename=Basis_V5_scaled.stl scale=0.00100000 0.00100000 0.0010000
